File: m5-atom-carrier-board.kicad_pcb (KiCad board)
At the start: 2 copper layers, 40 x 25 mm, 10 parts, among them J1 Grove, SW1 Button, U1 M5Atom

Commit message: minor adjustments
Other:
- board text added: "locked"
- board text removed: "0x76656e"
- board text removed: "3V3"
- board text removed: "GND"
- board text removed: "LED"
- board text removed: "M5Atom WiFi Config Board V0.1"
- board text removed: "Switch"
- board text removed: "Vcc"
Changed lines of the file:
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@@
       (net 6 "+3V3") (pintype "passive") (thermal_bridge_angle 45))
   )
-  (footprint "Logo:Cat1-Logo_15x8.7mm_SilkScreen" (layer "B.Cu")
+  (footprint "Logo:Cat1-Logo_15x8.7mm_SilkScreen" locked (layer "B.Cu")
     (at 108.8 70.5 180)
     (fp_text reference "REF**" (at 0 3 unlocked) (layer "B.SilkS") hide
@@
       (stroke (width 0) (type solid)) (fill solid) (layer "B.SilkS"))
   )
-  (gr_rect (start 85.7 58.425) (end 94.2 66.375)
+  (gr_rect locked (start 85.7 58.425) (end 94.2 66.375)
     (stroke (width 0.1) (type default)) (fill none) (layer "B.SilkS"))
   (gr_arc locked (start 120 72) (mid 119.12132 74.12132) (end 117 75)
@@
   (gr_line locked (start 117 50) (end 83 50)
     (stroke (width 0.1) (type default)) (layer "Edge.Cuts"))
-  (gr_text "GND" (at 113.98 54.664) (layer "B.SilkS" knockout)
+  (gr_text locked "GND" (at 113.98 54.664) (layer "B.SilkS" knockout)
     (effects (font (size 1 1) (thickness 0.2) bold) (justify left bottom mirror))
   )
-  (gr_text "Vcc" (at 113.89 56.664) (layer "B.SilkS" knockout)
+  (gr_text locked "Vcc" (at 113.89 56.664) (layer "B.SilkS" knockout)
     (effects (font (size 1 1) (thickness 0.2) bold) (justify left bottom mirror))
   )
-  (gr_text "LED" (at 114.03 58.664) (layer "B.SilkS" knockout)
+  (gr_text locked "LED" (at 114.03 58.664) (layer "B.SilkS" knockout)
     (effects (font (size 1 1) (thickness 0.2) bold) (justify left bottom mirror))
   )
-  (gr_text "M5Atom\nWiFi\nConfig\nBoard V0.1" (at 94.2 64.625) (layer "B.SilkS" knockout)
+  (gr_text locked "M5Atom\nWiFi\nConfig\nBoard V0.1" (at 94.2 64.625) (layer "B.SilkS" knockout)
     (effects (font (size 1 1) (thickness 0.2) bold) (justify left bottom mirror))
   )
-  (gr_text "Switch" (at 113.98 60.664) (layer "B.SilkS" knockout)
+  (gr_text locked "Switch" (at 113.98 60.664) (layer "B.SilkS" knockout)
     (effects (font (size 1 1) (thickness 0.2) bold) (justify left bottom mirror))
   )
-  (gr_text "0x76656e" (at 94.2 66.135) (layer "B.SilkS")
+  (gr_text locked "0x76656e" (at 94.2 66.135) (layer "B.SilkS")
     (effects (font (size 1 1) (thickness 0.2) bold) (justify left bottom mirror))
   )
-  (gr_text "3V3" (at 96.916 66 270) (layer "F.SilkS" knockout)
+  (gr_text locked "3V3" (at 96.916 66 270) (layer "F.SilkS" knockout)
     (effects (font (size 1 1) (thickness 0.2) bold) (justify left bottom))
   )
-  (gr_text "LED" (at 91.836 55.97 270) (layer "F.SilkS" knockout)
+  (gr_text locked "LED" (at 91.836 55.97 270) (layer "F.SilkS" knockout)
     (effects (font (size 1 1) (thickness 0.2) bold) (justify left bottom))
   )
-  (gr_text "GND" (at 86.756 55.97 270) (layer "F.SilkS" knockout)
+  (gr_text locked "GND" (at 86.756 55.97 270) (layer "F.SilkS" knockout)
     (effects (font (size 1 1) (thickness 0.2) bold) (justify left bottom))
   )
-  (gr_text "Switch" (at 94.376 56.02 270) (layer "F.SilkS" knockout)
+  (gr_text locked "Switch" (at 94.376 56.02 270) (layer "F.SilkS" knockout)
     (effects (font (size 1 1) (thickness 0.2) bold) (justify left bottom))
   )
@@
   (segment (start 115 60) (end 112.414214 60) (width 0.25) (layer "F.Cu") (net 3))
   (segment (start 97.455534 52.464466) (end 95.04 54.88) (width 0.25) (layer "F.Cu") (net 3))
+  (segment (start 113.15 71.1) (end 113.15 64.9) (width 0.25) (layer "F.Cu") (net 3))
   (segment (start 113.5 51) (end 100.991068 51) (width 0.25) (layer "F.Cu") (net 3))
-  (segment (start 113.15 64.9) (end 113.15 71.1) (width 0.25) (layer "F.Cu") (net 3))
   (segment (start 111.707107 60.292893) (end 111 61) (width 0.25) (layer "F.Cu") (net 3))
   (segment (start 115 60) (end 115 60.978932) (width 0.25) (layer "F.Cu") (net 3))
@@
   (segment (start 111 64) (end 111 65.5) (width 0.25) (layer "F.Cu") (net 5))
   (via (at 111 65.5) (size 0.8) (drill 0.4) (layers "F.Cu" "B.Cu") (net 5))
-  (segment (start 115.62132 64.27868) (end 115.278679 64.621321) (width 0.25) (layer "B.Cu") (net 5))
-  (segment (start 116.5 58.742641) (end 116.5 62.157359) (width 0.25) (layer "B.Cu") (net 5))
-  (segment (start 113.157359 65.5) (end 111 65.5) (width 0.25) (layer "B.Cu") (net 5))
-  (segment (start 115.62132 56.62132) (end 115 56) (width 0.25) (layer "B.Cu") (net 5))
-  (arc (start 116.5 58.742641) (mid 116.271638 57.59459) (end 115.62132 56.62132) (width 0.25) (layer "B.Cu") (net 5))
-  (arc (start 115.278679 64.621321) (mid 114.305409 65.271639) (end 113.157359 65.5) (width 0.25) (layer "B.Cu") (net 5))
-  (arc (start 116.5 62.157359) (mid 116.271638 63.30541) (end 115.62132 64.27868) (width 0.25) (layer "B.Cu") (net 5))
+  (segment (start 115 56) (end 115.62132 56.62132) (width 0.25) (layer "B.Cu") (net 5))
+  (segment (start 116.5 58.742641) (end 116.5 62.5) (width 0.25) (layer "B.Cu") (net 5))
+  (segment (start 113.5 65.5) (end 111 65.5) (width 0.25) (layer "B.Cu") (net 5))
+  (arc (start 116.5 62.5) (mid 115.62132 64.62132) (end 113.5 65.5) (width 0.25) (layer "B.Cu") (net 5))
+  (arc (start 115.62132 56.62132) (mid 116.271625 57.594593) (end 116.5 58.742641) (width 0.25) (layer "B.Cu") (net 5))
   (segment (start 107.975 71.5) (end 107.975 68.439214) (width 0.25) (layer "F.Cu") (net 6))
   (segment (start 112.378932 73.5) (end 109.975 73.5) (width 0.25) (layer "F.Cu") (net 6))
@@
     )
   )
-  (group "" (id 45b56925-17f9-4c2b-a4f4-8e9f3d7b2573)
+  (group "" locked (id 45b56925-17f9-4c2b-a4f4-8e9f3d7b2573)
     (members
       2aa55392-f859-4cfc-8aea-2677c5ebeaf0
@@
     )
   )
-  (group "" (id 7f76fb73-7c54-4146-a75d-18bb298e8f8d)
+  (group "" locked (id 7f76fb73-7c54-4146-a75d-18bb298e8f8d)
     (members
       45b56925-17f9-4c2b-a4f4-8e9f3d7b2573
